Commit message: second update

File: src/f1tenth_description/urdf/f1tenth.xacro (robot description, xacro)
@@ -4,4 +4,5 @@
   <gazebo>
     <plugin name="gazebo_ros_control" filename="libgazebo_ros_control.so">
+      <!--robotNamespace>/f1tenth</robotNamespace-->
       <robotSimType>gazebo_ros_control/DefaultRobotHWSim</robotSimType>
     </plugin>
@@ -31,5 +32,5 @@
       <origin xyz="0 0 0.07" rpy=" 0 0 0"/>
       <geometry>
-        <box size=".4 .15 .05"/>
+        <box size=".4 .2 .07"/>
       </geometry>
       <material name="blue" />
@@ -63,8 +64,8 @@
     <inertial>
       <origin xyz="0 0 0" rpy="0 0 0" />
-      <mass value="0.44055" />
-      <inertia ixx="0.00026046" ixy="0"  ixz="0"
-               iyy="0.00026046" iyz="0"
-               izz="0.00041226" />
+      <mass value="0.29" />
+      <inertia ixx="0.0027" ixy="0"  ixz="0"
+               iyy="0.0027" iyz="0"
+               izz="0.001111" />
       </inertial>
   </link>
@@ -111,8 +112,8 @@
     <inertial>
       <origin xyz="0 0 0" rpy="0 0 0" />
-      <mass value="0.44055" />
-      <inertia ixx="0.00026046" ixy="0" ixz="0"
-               iyy="0.00026046" iyz="0"
-               izz="0.00041226" />
+      <mass value="0.29" />
+      <inertia ixx="0.0027" ixy="0"  ixz="0"
+               iyy="0.0027" iyz="0"
+               izz="0.001111" />
     </inertial>
   </link>
@@ -150,5 +151,5 @@
     <parent link="chassis" />
     <child link="left_steering_link" />
-    <axis xyz="0 0 -1" />
+    <axis xyz="0 0 1" />
     <limit effort="10" lower="-0.08" upper="0.08" velocity="0.5" />
   </joint>
@@ -171,5 +172,5 @@
     <parent link="chassis" />
     <child link="right_steering_link" />
-    <axis xyz="0 0 -1" />
+    <axis xyz="0 0 1" />
     <limit effort="10" lower="-0.08" upper="0.08" velocity="0.5" />
   </joint>
@@ -201,8 +202,8 @@
     <inertial>
       <origin xyz="0 0 0" rpy="0 0 0" />
-      <mass value="0.34055" />
-      <inertia ixx="0.00026046" ixy="0"  ixz="0"
-               iyy="0.00026046" iyz="0"
-               izz="0.00041226" />
+      <mass value="0.29" />
+      <inertia ixx="0.0027" ixy="0"  ixz="0"
+               iyy="0.0027" iyz="0"
+               izz="0.001111" />
     </inertial>
   </link>
@@ -249,8 +250,8 @@
     <inertial>
       <origin xyz="0 0 0" rpy="0 0 0" />
-      <mass value="0.34055" />
-      <inertia ixx="0.00026046" ixy="0" ixz="0"
-               iyy="0.00026046" iyz="0"
-               izz="0.00041226" />
+      <mass value="0.29" />
+      <inertia ixx="0.0027" ixy="0"  ixz="0"
+               iyy="0.0027" iyz="0"
+               izz="0.001111" />
     </inertial>
   </link>

Commit message: third update

File: src/f1tenth_description/urdf/f1tenth.xacro (robot description, xacro)
@@ -1,5 +1,5 @@
 <?xml version="1.0"?>
 <robot name="f1tenth" xmlns:xacro="http://www.ros.org/wiki/xacro">
-  <!-- ros_control plugin -->
+<!-- ros_control plugin -->
   <gazebo>
     <plugin name="gazebo_ros_control" filename="libgazebo_ros_control.so">
@@ -7,4 +7,76 @@
       <robotSimType>gazebo_ros_control/DefaultRobotHWSim</robotSimType>
     </plugin>
+  </gazebo>
+<!-- hokuyo -->
+  <gazebo reference="laser">
+    <material>Gazebo/Grey</material>
+    <sensor type="ray" name="hokuyo_sensor">
+      <pose>0 0 0.0124 0 0 0</pose>
+      <visualize>true</visualize>
+      <update_rate>40</update_rate>
+      <ray>
+        <scan>
+          <horizontal>
+            <samples>1081</samples>
+            <resolution>1</resolution>
+            <min_angle>-2.0943951023931953</min_angle>
+            <max_angle>2.0943951023931953</max_angle>
+          </horizontal>
+        </scan>
+        <range>
+          <min>0.10</min>
+          <max>10.0</max>
+          <resolution>0.01</resolution>
+        </range>
+        <noise>
+          <mean>0.0</mean>
+          <stddev>0.01</stddev>
+        </noise>
+      </ray>
+      <plugin name="gazebo_ros_hokuyo_controller" filename="libgazebo_ros_laser.so">
+        <topicName>/scan</topicName>
+        <frameName>laser</frameName>
+      </plugin>
+    </sensor>
+  </gazebo>
+<!-- camera -->
+  <gazebo reference="camera_link">
+    <sensor type="camera" name="camera1">
+      <update_rate>30.0</update_rate>
+      <camera name="head">
+        <horizontal_fov>1.3962634</horizontal_fov>
+        <image>
+          <width>800</width>
+          <height>800</height>
+          <format>R8G8B8</format>
+        </image>
+        <clip>
+          <near>0.02</near>
+          <far>300</far>
+        </clip>
+        <noise>
+          <type>gaussian</type>
+          <!-- Noise is sampled independently per pixel on each frame.
+               That pixel's noise value is added to each of its color
+               channels, which at that point lie in the range [0,1]. -->
+          <mean>0.0</mean>
+          <stddev>0.007</stddev>
+        </noise>
+      </camera>
+      <plugin name="camera_controller" filename="libgazebo_ros_camera.so">
+        <alwaysOn>true</alwaysOn>
+        <updateRate>0.0</updateRate>
+        <cameraName>f1tenth/camera</cameraName>
+        <imageTopicName>image_raw</imageTopicName>
+        <cameraInfoTopicName>camera_info</cameraInfoTopicName>
+        <frameName>camera_link</frameName>
+        <hackBaseline>0.07</hackBaseline>
+        <distortionK1>0.0</distortionK1>
+        <distortionK2>0.0</distortionK2>
+        <distortionK3>0.0</distortionK3>
+        <distortionT1>0.0</distortionT1>
+        <distortionT2>0.0</distortionT2>
+      </plugin>
+    </sensor>
   </gazebo>
 <!-- Import Rviz colors -->
@@ -25,5 +97,5 @@
       <origin xyz="0 0 0.07" rpy=" 0 0 0"/>
       <geometry>
-        <box size=".4 .2 .05"/>
+        <box size=".4 .2 .08"/>
       </geometry>
       <material name="blue" />
@@ -152,5 +224,5 @@
     <child link="left_steering_link" />
     <axis xyz="0 0 1" />
-    <limit effort="10" lower="-0.08" upper="0.08" velocity="0.5" />
+    <limit effort="10" lower="-0.5" upper="0.5" velocity="0.5" />
   </joint>
   <transmission name="left_steering_trans">
@@ -173,5 +245,5 @@
     <child link="right_steering_link" />
     <axis xyz="0 0 1" />
-    <limit effort="10" lower="-0.08" upper="0.08" velocity="0.5" />
+    <limit effort="10" lower="-0.5" upper="0.5" velocity="0.5" />
   </joint>
   <transmission name="right_steering_trans">
@@ -293,3 +365,59 @@
     <material>Gazebo/Orange</material>
   </gazebo>
+  <!-- Add Hokuyo laser scanner -->
+  <link name="laser">
+    <inertial>
+        <origin xyz="0 0 0" rpy="0 0 0" />
+	    <mass value="0.130" />
+	    <inertia ixx="4E-06" ixy="0" ixz="0"
+		     iyy="4E-06" iyz="0"
+		     izz="4E-06" />
+    </inertial>
+    <collision>
+      <origin xyz="0 0 0" rpy="0 0 0"/>
+      <geometry>
+        <box size="0.1 0.1 0.1"/>
+      </geometry>
+    </collision>
+    <visual>
+      <origin xyz="0 0 0" rpy="0 0 0"/>
+      <geometry>
+        <mesh filename="package://f1tenth_description/meshes/hokuyo.dae"/>
+        <material name="grey" />
+      </geometry>
+    </visual>
+  </link>
+  <joint name="hokuyo_joint" type="fixed">
+    <origin xyz="-0.1 0 0.12" rpy="0 0 0"/>
+    <parent link="chassis" />
+    <child link="laser" />
+    <axis xyz="0 0 1" />
+  </joint>
+<!-- Camera -->
+  <link name="camera_link">
+    <collision>
+      <origin xyz="0 0 0" rpy="0 0 0"/>
+      <geometry>
+    <box size=" 0.02 0.1 0.02"/>
+      </geometry>
+    </collision>
+    <visual>
+      <origin xyz="0 0 0" rpy="0 0 0"/>
+      <geometry>
+        <box size="0.02 0.1 0.02"/>
+      </geometry>
+      <material name="blue"/>
+    </visual>
+    <inertial>
+      <mass value="1e-5" />
+      <origin xyz="0 0 0" rpy="0 0 0"/>
+      <inertia ixx="1e-6" ixy="0" ixz="0" iyy="1e-6" iyz="0" izz="1e-6" />
+    </inertial>
+  </link>
+  <joint name="camera_joint" type="fixed">
+    <axis xyz="0 1 0" />
+    <origin xyz="0.208 0 0.1" rpy="0 0 0"/>
+    <parent link="chassis"/>
+    <child link="camera_link"/>
+  </joint>
 </robot>

Commit message: third update

File: src/f1tenth_description/urdf/f1tenth.xacro (robot description, xacro)
@@ -42,41 +42,55 @@
 <!-- camera -->
   <gazebo reference="camera_link">
-    <sensor type="camera" name="camera1">
-      <update_rate>30.0</update_rate>
-      <camera name="head">
-        <horizontal_fov>1.3962634</horizontal_fov>
-        <image>
-          <width>800</width>
-          <height>800</height>
-          <format>R8G8B8</format>
-        </image>
-        <clip>
-          <near>0.02</near>
-          <far>300</far>
-        </clip>
-        <noise>
-          <type>gaussian</type>
-          <!-- Noise is sampled independently per pixel on each frame.
-               That pixel's noise value is added to each of its color
-               channels, which at that point lie in the range [0,1]. -->
-          <mean>0.0</mean>
-          <stddev>0.007</stddev>
-        </noise>
-      </camera>
-      <plugin name="camera_controller" filename="libgazebo_ros_camera.so">
-        <alwaysOn>true</alwaysOn>
-        <updateRate>0.0</updateRate>
-        <cameraName>f1tenth/camera</cameraName>
-        <imageTopicName>image_raw</imageTopicName>
-        <cameraInfoTopicName>camera_info</cameraInfoTopicName>
-        <frameName>camera_link</frameName>
-        <hackBaseline>0.07</hackBaseline>
-        <distortionK1>0.0</distortionK1>
-        <distortionK2>0.0</distortionK2>
-        <distortionK3>0.0</distortionK3>
-        <distortionT1>0.0</distortionT1>
-        <distortionT2>0.0</distortionT2>
-      </plugin>
+    <sensor type="depth" name="camera1">
+        <always_on>1</always_on>
+        <visualize>true</visualize>
+        <camera>
+            <horizontal_fov>1.047</horizontal_fov>
+            <image>
+                <width>640</width>
+                <height>480</height>
+                <format>R8G8B8</format>
+            </image>
+            <depth_camera>
+            </depth_camera>
+            <clip>
+                <near>0.1</near>
+                <far>100</far>
+            </clip>
+        </camera>
+             <plugin name="camera_controller" filename="libgazebo_ros_openni_kinect.so">
+             <alwaysOn>true</alwaysOn>
+                <updateRate>10.0</updateRate>
+                <cameraName>camera</cameraName>
+                <frameName>camera_link</frameName>
+            <imageTopicName>rgb/image_raw</imageTopicName>
+            <depthImageTopicName>depth/image_raw</depthImageTopicName>
+            <pointCloudTopicName>depth/points</pointCloudTopicName>
+            <cameraInfoTopicName>rgb/camera_info</cameraInfoTopicName>
+            <depthImageCameraInfoTopicName>depth/camera_info</depthImageCameraInfoTopicName>
+            <pointCloudCutoff>0.4</pointCloudCutoff>
+                <hackBaseline>0.07</hackBaseline>
+                <distortionK1>0.0</distortionK1>
+                <distortionK2>0.0</distortionK2>
+                <distortionK3>0.0</distortionK3>
+                <distortionT1>0.0</distortionT1>
+                <distortionT2>0.0</distortionT2>
+            <CxPrime>0.0</CxPrime>
+            <Cx>0.0</Cx>
+            <Cy>0.0</Cy>
+            <focalLength>0.0</focalLength>
+            </plugin>
     </sensor>
+  </gazebo>
+<!--IMU-->
+  <gazebo>
+    <plugin name="imu_plugin" filename="libgazebo_ros_imu.so">
+      <alwaysOn>true</alwaysOn>
+      <bodyName>imu_link</bodyName>
+      <topicName>imu</topicName>
+      <serviceName>imu_service</serviceName>
+      <gaussianNoise>0.0</gaussianNoise>
+      <updateRate>20.0</updateRate>
+    </plugin>
   </gazebo>
 <!-- Import Rviz colors -->
@@ -421,3 +435,13 @@
     <child link="camera_link"/>
   </joint>
+<!--IMU-->
+  <link name="imu_link">
+    <xacro:null_inertial/>
+  </link>
+  <joint name="imu_joint" type="fixed">
+    <axis xyz="0 1 0" />
+    <origin xyz="0 0 0.1" rpy="0 0 0"/>
+    <parent link="chassis"/>
+    <child link="imu_link"/>
+  </joint>
 </robot>
